Commit message: updates

File: my_box_bot_gazebo/urdf/Assem1_urdf.urdf (robot description, URDF)
Before this commit: robot design1_urdf, 9 links, 8 joints
Links:
- link acc1: mass 0.580805573043355 -> 0.580805573043362; geometry collision mesh filename=package://Assem1_urdf/meshes/acc1.STL; visual mesh filename=package://Assem1_urdf/meshes/acc1.STL
- link acc2: geometry collision mesh filename=package://Assem1_urdf/meshes/acc2.STL; visual mesh filename=package://Assem1_urdf/meshes/acc2.STL
- link base_link: geometry collision mesh filename=package://Assem1_urdf/meshes/base_link.STL; visual mesh filename=package://Assem1_urdf/meshes/base_link.STL
- link cbracket: geometry collision mesh filename=package://Assem1_urdf/meshes/cbracket.STL; visual mesh filename=package://Assem1_urdf/meshes/cbracket.STL
- link leg1: geometry collision mesh filename=package://Assem1_urdf/meshes/leg1.STL; visual mesh filename=package://Assem1_urdf/meshes/leg1.STL
- link leg2: geometry collision mesh filename=package://Assem1_urdf/meshes/leg2.STL; visual mesh filename=package://Assem1_urdf/meshes/leg2.STL
- link lowleg1: geometry collision mesh filename=package://Assem1_urdf/meshes/lowleg1.STL; visual mesh filename=package://Assem1_urdf/meshes/lowleg1.STL
- link lowleg2: geometry collision mesh filename=package://Assem1_urdf/meshes/lowleg2.STL; visual mesh filename=package://Assem1_urdf/meshes/lowleg2.STL
- link pulley: geometry collision mesh filename=package://Assem1_urdf/meshes/pulley.STL; visual mesh filename=package://Assem1_urdf/meshes/pulley.STL
Joints:
- joint j1: axis 0 0 1 -> 0 0 -1
